File: clock/clock.kicad_pcb (KiCad board)
At the start: 4 copper layers, 31 parts, among them J1 LED_connector

Commit message: finished LED digit PCB, added gerber files, moved microcontroller kicad pcb files to different directory
Parts:
- removed D10, D11, D12, D13, D14, D15, D16, D17, D18, D19, D20, D21, D22, D23, D24, D25, D26, D27, D28, D29, D30: WS2812B, LED_SMD:oneLED
- added G***: LOGO, LOGO, B.Cu at (215.4, 130.0)
- added J5: LED_connector, Connector_PinHeader_2.54mm:PinHeader_1x03_P2.54mm_Vertical, F.Cu at (218.0, 157.5)
- added J6: LED_connector, Connector_PinHeader_2.54mm:PinHeader_1x03_P2.54mm_Vertical, F.Cu at (225.6, 157.5)
- added J7: LED_connector, Connector_PinHeader_2.54mm:PinHeader_1x03_P2.54mm_Vertical, F.Cu at (251.9, 157.5)
- added mouse-bite-2mm-slot: VAL**, Panelization.pretty-master:mouse-bite-2mm-slot, F.Cu at (164.3, 118.0)
- added mouse-bite-2mm-slot1: VAL**, Panelization.pretty-master:mouse-bite-2mm-slot, F.Cu at (181.6, 118.0)
- added mouse-bite-2mm-slot10: VAL**, Panelization.pretty-master:mouse-bite-2mm-slot, F.Cu at (247.2, 202.0)
- added mouse-bite-2mm-slot11: VAL**, Panelization.pretty-master:mouse-bite-2mm-slot, F.Cu at (221.8, 141.3)
- added mouse-bite-2mm-slot12: VAL**, Panelization.pretty-master:mouse-bite-2mm-slot, F.Cu at (221.8, 158.6)
- added mouse-bite-2mm-slot13: VAL**, Panelization.pretty-master:mouse-bite-2mm-slot, F.Cu at (221.8, 175.9)
- added mouse-bite-2mm-slot14: VAL**, Panelization.pretty-master:mouse-bite-2mm-slot, F.Cu at (221.8, 193.2)
- added mouse-bite-2mm-slot2: VAL**, Panelization.pretty-master:mouse-bite-2mm-slot, F.Cu at (198.9, 118.0)
- added mouse-bite-2mm-slot3: VAL**, Panelization.pretty-master:mouse-bite-2mm-slot, F.Cu at (229.9, 118.0)
- added mouse-bite-2mm-slot3: VAL**, Panelization.pretty-master:mouse-bite-2mm-slot, F.Cu at (216.2, 118.0)
- added mouse-bite-2mm-slot3: VAL**, Panelization.pretty-master:mouse-bite-2mm-slot, F.Cu at (221.8, 124.0)
- added mouse-bite-2mm-slot4: VAL**, Panelization.pretty-master:mouse-bite-2mm-slot, F.Cu at (164.3, 202.0)
- added mouse-bite-2mm-slot5: VAL**, Panelization.pretty-master:mouse-bite-2mm-slot, F.Cu at (181.6, 202.0)
- added mouse-bite-2mm-slot6: VAL**, Panelization.pretty-master:mouse-bite-2mm-slot, F.Cu at (198.9, 202.0)
- added mouse-bite-2mm-slot7: VAL**, Panelization.pretty-master:mouse-bite-2mm-slot, F.Cu at (216.2, 202.0)
- added mouse-bite-2mm-slot8: VAL**, Panelization.pretty-master:mouse-bite-2mm-slot, F.Cu at (247.2, 118.0)
- added mouse-bite-2mm-slot9: VAL**, Panelization.pretty-master:mouse-bite-2mm-slot, F.Cu at (229.9, 202.0)
- moved J1 117.7 mm to (162.4, 157.5), turned to 0 degrees
- moved D9 113.3 mm to (244.3, 152.8), turned to 90 degrees
- moved D2 99.6 mm to (178.4, 185.3), turned to 90 degrees
- moved D3 98.5 mm to (178.4, 151.8), turned to 90 degrees
- moved D5 93.7 mm to (201.9, 134.8), turned to -90 degrees
- moved D7 93.5 mm to (201.9, 168.3), turned to -90 degrees
- moved D8 87.6 mm to (244.3, 186.3), turned to 90 degrees
- moved D4 85.5 mm to (181.7, 131.4)
- moved D6 85.5 mm to (181.7, 164.9)
- moved D1 85.0 mm to (181.7, 198.4)
Connections:
- D1 pad 4: Net-(D1-DIN) -> D_In1
- D2 pad 4: D_In -> Net-(D1-DOUT)
- D4 pad 2: Net-(D1-DIN) -> Net-(D4-DOUT)
- D4 pad 4: Net-(D4-DIN) -> Net-(D3-DOUT)
- D5 pad 2: Net-(D10-DIN) -> Net-(D5-DOUT)
- D5 pad 4: Net-(D12-DOUT) -> Net-(D4-DOUT)
- D6 pad 2: Net-(D14-DIN) -> Net-(D6-DOUT)
- D6 pad 4: Net-(D1-DOUT) -> Net-(D5-DOUT)
- D7 pad 2: Net-(D13-DIN) -> D_Out1
- D7 pad 4: Net-(D3-DOUT) -> Net-(D6-DOUT)
- D8 pad 1: 5V -> 5V2
- D8 pad 2: Net-(D11-DIN) -> Net-(D8-DOUT)
- D8 pad 4: Net-(D14-DOUT) -> D_In2
- D9 pad 1: 5V -> 5V2
- D9 pad 2: Net-(D4-DIN) -> D_Out2
- D9 pad 4: Net-(D10-DOUT) -> Net-(D8-DOUT)
- J1 pad 2: D_In -> D_In1
Routing:
- net D_In1: track 0.00 -> 49.6 mm, vias 0 -> 2
- net Net-(D1-DOUT): track 0.00 -> 45.5 mm, vias 0 -> 2
- net D_Out1: track 0.00 -> 44.6 mm, vias 0 -> 2
- net D_In2: track 0.00 -> 42.8 mm, vias 0 -> 2
- net D_Out2: track 0.00 -> 37.7 mm, vias 0 -> 2
- net Net-(D5-DOUT): track 0.00 -> 37.5 mm, vias 0 -> 2
- net GND: track 0.00 -> 28.1 mm, vias 0 -> 9
- net 5V: track 0.00 -> 20.8 mm, vias 0 -> 7
- net Net-(D8-DOUT): track 0.00 -> 19.0 mm, vias 0 -> 4
- net Net-(D2-DOUT): track 0.00 -> 19.0 mm, vias 0 -> 2
- net Net-(D3-DOUT): track 0.00 -> 15.8 mm, vias 0 -> 2
- net Net-(D6-DOUT): track 0.00 -> 15.5 mm, vias 0 -> 2
- net Net-(D4-DOUT): track 0.00 -> 14.4 mm, vias 0 -> 2
- net 5V2: track 0.00 -> 9.02 mm, vias 0 -> 2
- added copper zone on In2.Cu, net 5V
- added copper zone on In2.Cu, net 5V2
- added copper zone on In1.Cu, net GND
Other:
- board outline added: 95.1 x 102 mm
- board text added: "Designed by Henry To June 19th, 2025 Digital Clock Digit"
- board text added: "Digital Clock Delimiter"
