File: clock/clock.kicad_sch (KiCad schematic)
At the start: 31 parts, among them J1 LED_connector

Commit message: finished LED digit PCB, added gerber files, moved microcontroller kicad pcb files to different directory
Parts:
- removed D10, D11, D12, D13, D14, D15, D16, D17, D18, D19, D20, D21, D22, D23, D24, D25, D26, D27, D28, D29, D30: WS2812B, LED_SMD:oneLED, symbol LED:WS2812B
- added J5: male_connector, Connector_PinHeader_2.54mm:PinHeader_1x03_P2.54mm_Vertical, symbol Connector_Generic:Conn_01x03
- added J6: female connector, Connector_PinHeader_2.54mm:PinHeader_1x03_P2.54mm_Vertical, symbol Connector_Generic:Conn_01x03
- added J7: male connector, Connector_PinHeader_2.54mm:PinHeader_1x03_P2.54mm_Vertical, symbol Connector_Generic:Conn_01x03
- J1: value LED_connector -> female_connector
Connections:
- net 5V: now also J5.3 (Pin_3); no longer D8.1 (VDD), D9.1 (VDD)
- net GND: now also J5.1 (Pin_1), J6.1 (Pin_1), J7.1 (Pin_1)
- net at D4.4 (DIN): now also D3.2 (DOUT); no longer D9.2 (DOUT)
- net at D9.4 (DIN): now also D8.2 (DOUT)
- net at D6.2 (DOUT): now also D7.4 (DIN)
- net at D1.2 (DOUT): now also D2.4 (DIN); no longer D6.4 (DIN)
- net at D4.2 (DOUT): now also D5.4 (DIN); no longer D1.4 (DIN)
- net D_Out1: now reaches D7.2 (DOUT)
- net D_Out1: now also J5.2 (Pin_2)
- net D_In2: now reaches D8.4 (DIN)
- net D_In2: now also J6.2 (Pin_2)
- net at D5.2 (DOUT): now also D6.4 (DIN)
- net D_In renamed D_In1
- net D_In1: now also D1.4 (DIN); no longer D2.4 (DIN)
- new net 5V2: D8.1 (VDD), D9.1 (VDD), J6.3 (Pin_3), J7.3 (Pin_3)
- new net D_Out2: D9.2 (DOUT), J7.2 (Pin_2)
- no-connect marks 1 -> 0
Other:
- removed sheet digiClockMicro
- note added: "Individual Digit LED setup"
- note added: "LED delimiter setup"
- moved on the sheet: J1
